Commit message: Update tetraDS.xacro

File: tetraDS_description/urdf/tetraDS/tetraDS.xacro (robot description, xacro)
@@ -28,6 +28,5 @@
   </link>
   <joint name="laser_flag" type="fixed">
-    <!--<origin xyz="0.1372 0 0.142" rpy="0 0 0" />-->
-    <origin xyz="0.1372 0 -0.00636" rpy="3.14 0 0" />
+    <origin xyz="0.1372 0 0.142" rpy="0 0 0" />
     <parent link="base_link"/>
     <child link="laser" />
@@ -141,6 +140,5 @@
   </link>
   <joint name="camera1_link" type="fixed">
-    <!--<origin xyz="0.1553 -0.1155 0.0" rpy="3.14 -0.261799 0" />-->
-    <origin xyz="0.1553 -0.079 0.0" rpy="0 -0.261799 0" />
+    <origin xyz="0.1553 -0.079 0.0" rpy="0 0 0" />
     <parent link="base_link"/>
     <child link="camera1_link" />
@@ -156,5 +154,5 @@
   </link>
   <joint name="camera2_link" type="fixed">
-    <origin xyz="0.1553 0.1145 0.0" rpy="0 -0.261799 0" />
+    <origin xyz="0.1553 0.1145 0.0" rpy="0 0 0" />
     <parent link="base_link"/>
     <child link="camera2_link" />

Commit message: Update tetraDS.xacro

File: tetraDS_description/urdf/tetraDS/tetraDS.xacro (robot description, xacro)
@@ -140,5 +140,5 @@
   </link>
   <joint name="camera1_link" type="fixed">
-    <origin xyz="0.1553 -0.079 0.0" rpy="0 0 0" />
+    <origin xyz="0.1553 0.079 0.0" rpy="0 0 0" />
     <parent link="base_link"/>
     <child link="camera1_link" />
@@ -154,5 +154,5 @@
   </link>
   <joint name="camera2_link" type="fixed">
-    <origin xyz="0.1553 0.1145 0.0" rpy="0 0 0" />
+    <origin xyz="0.1553 -0.1145 0.0" rpy="0 0 0" />
     <parent link="base_link"/>
     <child link="camera2_link" />

Commit message: Update tetraDS.xacro

File: tetraDS_description/urdf/tetraDS/tetraDS.xacro (robot description, xacro)
@@ -140,5 +140,5 @@
   </link>
   <joint name="camera1_link" type="fixed">
-    <origin xyz="0.1553 0.079 0.0" rpy="0 0 0" />
+    <origin xyz="0.1553 -0.079 0.0" rpy="0 0 0" />
     <parent link="base_link"/>
     <child link="camera1_link" />
@@ -154,5 +154,5 @@
   </link>
   <joint name="camera2_link" type="fixed">
-    <origin xyz="0.1553 -0.1145 0.0" rpy="0 0 0" />
+    <origin xyz="0.1553 0.1145 0.0" rpy="0 0 0" />
     <parent link="base_link"/>
     <child link="camera2_link" />
